File: v1_0/KiCad Schematic.kicad_pcb (KiCad board)
At the start: 2 copper layers, 50.1 x 70 mm, 81 parts, among them IC1 MC7805BDTRKG, IC2 ATSAMD51J19A-MU, J1 47309-3351, J10 Conn_01x04, J11 Conn_01x04, J12 Conn_01x03, J13 Conn_01x03, J14 Conn_01x20, J15 Conn_01x03, J16 Conn_01x03, J17 Hole, J18 Hole, J19 Hole, J2 Conn_01x02, J20 Hole, J21 Conn_01x02, J3 47346-0001, J4 Conn_01x04, J5 Conn_01x04, J6 20021121-00010C4LF, J7 Conn_01x02, J8 Conn_01x02, J9 Conn_01x02, Q1 NVTFS5C680NLTAG, Q2 NVTFS5C680NLTAG, U1 TMC2041-LA, U2 TMC2041-LA, U3 AP2112K-3.3, Y1 LFXTAL009678REEL

Commit message: v1.0 release
Parts:
- added D2: LED, LED_SMD:LED_0603_1608Metric, F.Cu at (61.5, 153.8)
- added D3: CGRTS4004-HF, Diode_SMD:D_SOD-123F, F.Cu at (25.7, 175.7)
- added D4: CGRTS4004-HF, Diode_SMD:D_SOD-123F, F.Cu at (31.9, 183.8)
- added G***: LOGO, imgs:smol_logo, F.Cu at (41.9, 151.3)
- added G***: LOGO, imgs:logo, B.Cu at (55.1, 171.6)
- added R16: 10k, Resistor_SMD:R_0603_1608Metric, F.Cu at (55.3, 151.7)
- added R18: 10k, Resistor_SMD:R_0603_1608Metric, F.Cu at (54.2, 152.9)
- added R19: 174, Resistor_SMD:R_0603_1608Metric, F.Cu at (34.6, 164.2)
- added R20: 174, Resistor_SMD:R_0603_1608Metric, F.Cu at (59.8, 153.8)
- C32, C33: value 22nF -> 22pF
- IC2: footprint SamacSys_Parts:QFN50P900X900X100-65N-D -> Package_DFN_QFN:QFN-64-1EP_9x9mm_P0.5mm_EP6x6mm_ThermalVias
- moved C3 9.53 mm to (33.0, 164.2), turned to 270 degrees
- moved R15 8.92 mm to (41.8, 171.7), turned to 180 degrees
- moved C12 2.90 mm to (37.8, 186.5)
- moved C13 2.90 mm to (37.8, 182.7)
- moved C16 2.90 mm to (45.8, 191.9)
- moved C19 2.90 mm to (51.9, 186.7)
- moved C20 2.90 mm to (57.5, 184.6)
- moved J10 2.90 mm to (49.1, 193.7)
- moved J11 2.90 mm to (41.9, 193.8)
- moved R4 2.90 mm to (37.6, 184.7)
- moved R5 2.90 mm to (52.1, 184.9)
- moved R6 2.90 mm to (37.6, 188.3)
- moved R7 2.90 mm to (52.1, 188.5)
- moved U2 2.90 mm to (44.9, 186.5)
- moved R13 2.22 mm to (29.9, 177.7)
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Connections:
- IC2 pad 10: /GEN0 -> /GATE0
- IC2 pad 11: /GEN1 -> /GATE1
- IC2 pad 12: /GEN2 -> /GEN0
- IC2 pad 13: /GEN3 -> /GEN1
- IC2 pad 14: /GEN4 -> /GEN2
- IC2 pad 15: /GEN5 -> /GEN3
- IC2 pad 16: /GEN6 -> /GEN4
- IC2 pad 17: /GEN7 -> /GEN5
- IC2 pad 18: /GEN8 -> /GEN6
- IC2 pad 19: /GEN9 -> /GEN7
- IC2 pad 20: /GEN10 -> /GEN8
- IC2 pad 23: /GEN11 -> /GEN9
- IC2 pad 24: /GEN12 -> /GEN10
- IC2 pad 25: /GEN13 -> /GEN11
- IC2 pad 26: /GEN14 -> /GEN12
- IC2 pad 27: /GEN15 -> /GEN13
- IC2 pad 28: /GEN16 -> /GEN14
- IC2 pad 59: /GATE1 -> /D0_EN
- IC2 pad 6: Net-(IC2-Pad6) -> /D0_S1_STEP
- IC2 pad 60: /GATE0 -> /D0_S0_STEP
- IC2 pad 61: /D0_EN -> /D0_S0_DIR
- IC2 pad 62: /D0_S0_STEP -> Net-(IC2-Pad62)
- IC2 pad 63: /D0_S0_DIR -> Net-(IC2-Pad63)
- IC2 pad 64: /D0_S1_STEP -> Net-(IC2-Pad64)
- J14 pad 1: /GEN0 -> /GATE0
- J14 pad 10: /GEN9 -> /GEN7
- J14 pad 11: /GEN10 -> /GEN8
- J14 pad 12: /GEN11 -> /GEN9
- J14 pad 13: /GEN12 -> /GEN10
- J14 pad 14: /GEN13 -> /GEN11
- J14 pad 15: /GEN14 -> /GEN12
- J14 pad 16: /GEN15 -> /GEN13
- J14 pad 17: /GEN16 -> /GEN14
- J14 pad 2: /GEN1 -> /GATE1
- J14 pad 3: /GEN2 -> /GEN0
- J14 pad 4: /GEN3 -> /GEN1
- J14 pad 5: /GEN4 -> /GEN2
- J14 pad 6: /GEN5 -> /GEN3
- J14 pad 7: /GEN6 -> /GEN4
- J14 pad 8: /GEN7 -> /GEN5
- J14 pad 9: /GEN8 -> /GEN6
- J6 pad 10: Net-(J6-Pad10) -> /RESET
- J6 pad 2: GND -> /SWDIO
- J6 pad 3: /SWDIO -> GND
- J6 pad 5: Net-(J6-Pad5) -> GND
- S1 pad 1: Net-(S1-Pad1) -> Net-(R19-Pad1)
- S1 pad 2: Net-(S1-Pad2) -> GND
- S1 pad 3: Net-(S1-Pad3) -> GND
- S1 pad 4: Net-(S1-Pad4) -> Net-(R19-Pad1)
- S1 pad 5: Net-(S1-Pad5) -> GND
Routing:
- net /GATE1: track 38.4 -> 83.7 mm, vias 0 -> 2
- net /GATE0: track 21.0 -> 65.6 mm, vias 0 -> 4
- net GND: track 196.6 -> 218.5 mm, vias 38 -> 30
- net /RESET: track 12.6 -> 33.8 mm
- net /GEN16: track 18.8 -> 0.00 mm
- net +3V3: track 235.3 -> 253.1 mm, vias 13 -> 14
- net /GEN15: track 17.0 -> 0.00 mm
- net Net-(R19-Pad1): track 0.00 -> 9.00 mm
- net Net-(D4-Pad2): track 8.28 -> 16.0 mm
- net /GEN14: track 16.2 -> 22.4 mm
- net +VDC: track 96.2 -> 101.3 mm, vias 15 -> 17
- net /D0_S1_STEP: track 16.3 -> 21.3 mm, vias 0 -> 2
- net /MOSI: track 163.7 -> 168.0 mm
- net /GEN3: track 20.1 -> 16.0 mm
- net /GEN2: track 22.4 -> 18.4 mm
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Other:
- board text added: ""I really like ceilings... I guess you could call me a ceiling fan" -Unknown"
- board text added: "1.0"
- board text added: "G0"
- board text added: "G1"
- board text added: "JLCJLCJLCJLC"
- board text added: "RX|TX"
- board text removed: "15"
- board text removed: "16"
- board text removed: "RX TX"
