File: v1_0/KiCad Schematic.sch (KiCad schematic (older format))
At the start: 81 parts, among them IC1 MC7805BDTRKG, IC2 ATSAMD51J19A-MU, J1 47309-3351, J10 Conn_01x04, J11 Conn_01x04, J12 Conn_01x03, J13 Conn_01x03, J14 Conn_01x20, J15 Conn_01x03, J16 Conn_01x03, J17 Hole, J18 Hole, J19 Hole, J2 Conn_01x02, J20 Hole, J21 Conn_01x02, J3 47346-0001, J4 Conn_01x04, J5 Conn_01x04, J6 20021121-00010C4LF, J7 Conn_01x02, J8 Conn_01x02, J9 Conn_01x02, Q1 NVTFS5C680NLTAG, Q2 NVTFS5C680NLTAG, U1 TMC2041-LA, U2 TMC2041-LA, U3 AP2112K-3.3, Y1 LFXTAL009678REEL

Commit message: v1.0 release
Parts:
- added D2: LED, LED_SMD:LED_0603_1608Metric, symbol Device:LED
- added D3, D4: CGRTS4004-HF, Diode_SMD:D_SOD-123F, symbol Device:D
- added R16, R18: 10k, Resistor_SMD:R_0603_1608Metric, symbol Device:R
- added R19, R20: 174, Resistor_SMD:R_0603_1608Metric, symbol Device:R
- C32, C33: value 22nF -> 22pF
- IC2: footprint QFN50P900X900X100-65N-D -> Package_DFN_QFN:QFN-64-1EP_9x9mm_P0.5mm_EP6x6mm_ThermalVias
Connections:
- net GEN15 is gone; now on net GEN13: IC2.27 (PB14), J14.16 (Pin_16)
- net GEN16 is gone; now on net GEN14: IC2.28 (PB15), J14.17 (Pin_17)
- net +3V3: now also R16.1, R18.1
- net +VDC: now also D3.1 (K), D4.1 (K)
- net D0_EN: now also IC2.59 (PB30); no longer IC2.61 (PB00)
- net D0_S0_DIR: now also IC2.61 (PB00); no longer IC2.63 (PB02)
- net D0_S0_STEP: now also IC2.60 (PB31); no longer IC2.62 (PB01)
- net D0_S1_STEP: now also IC2.6 (PB05); no longer IC2.64 (PB03)
- net GATE0: now also IC2.10 (PB07), J14.1 (Pin_1); no longer IC2.60 (PB31)
- net GATE1: now also IC2.11 (PB08), J14.2 (Pin_2); no longer IC2.59 (PB30)
- net GEN0: now also IC2.12 (PB09), J14.3 (Pin_3); no longer IC2.10 (PB07), J14.1 (Pin_1)
- net GEN1: now also IC2.13 (PA04), J14.4 (Pin_4); no longer IC2.11 (PB08), J14.2 (Pin_2)
- net GEN10: now also IC2.24 (PB11), J14.13 (Pin_13); no longer IC2.20 (PA11), J14.11 (Pin_11)
- net GEN11: now also IC2.25 (PB12), J14.14 (Pin_14); no longer IC2.23 (PB10), J14.12 (Pin_12)
- net GEN12: now also IC2.26 (PB13), J14.15 (Pin_15); no longer IC2.24 (PB11), J14.13 (Pin_13)
- net GEN13: no longer IC2.25 (PB12), J14.14 (Pin_14)
- net GEN14: now also R20.2; no longer IC2.26 (PB13), J14.15 (Pin_15)
- net GEN2: now also IC2.14 (PA05), J14.5 (Pin_5); no longer IC2.12 (PB09), J14.3 (Pin_3)
- net GEN3: now also IC2.15 (PA06), J14.6 (Pin_6); no longer IC2.13 (PA04), J14.4 (Pin_4)
- net GEN4: now also IC2.16 (PA07), J14.7 (Pin_7); no longer IC2.14 (PA05), J14.5 (Pin_5)
- net GEN5: now also IC2.17 (PA08), J14.8 (Pin_8); no longer IC2.15 (PA06), J14.6 (Pin_6)
- net GEN6: now also IC2.18 (PA09), J14.9 (Pin_9); no longer IC2.16 (PA07), J14.7 (Pin_7)
- net GEN7: now also IC2.19 (PA10), J14.10 (Pin_10); no longer IC2.17 (PA08), J14.8 (Pin_8)
- net GEN8: now also IC2.20 (PA11), J14.11 (Pin_11); no longer IC2.18 (PA09), J14.9 (Pin_9)
- net GEN9: now also IC2.23 (PB10), J14.12 (Pin_12); no longer IC2.19 (PA10), J14.10 (Pin_10)
- net GND: now also J6.3, J6.5, S1.2 (NO_1), S1.3 (NO_2), S1.5 (GND), D2.1 (K); no longer J6.2
- net RESET: now also J6.10, R19.2
- net SCL: now also R18.2
- net SDA: now also R16.2
- net SWDIO: now also J6.2; no longer J6.3
- net at J7.2 (Pin_2), Q1.5 (D_1), Q1.6 (D_2)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: now also D3.2 (A)
- net at J8.2 (Pin_2), Q2.5 (D_1), Q2.6 (D_2)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: now also D4.2 (A)
- net at S1.1 (COM_1): now also S1.4 (COM_2), R19.1
- new net: D2.2 (A), R20.1
Other:
- note added: "COMS I/O"
- note added: "FET GATES"
- note added: "GPIO"
- note added: "MCU"
- note added: "POWER FILTERING"
- note added: "POWER REG"
- note added: "PROG HEADER"
- note added: "STATUS"
- note added: "STEPPERS 0/1"
- note added: "STEPPERS 2/3\n"
- moved on the sheet: C1, C10, C11, C12, C13, C14, C15, C16, C17, C18, C19, C2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
