File: pcb/KiCad Schematic.sch (KiCad schematic (older format))
At the start: 88 parts, among them IC1 MC7805BDTRKG, IC2 ATSAMD51J19A-MU, J1 47309-3351, J10 Conn_01x04, J11 Conn_01x04, J12 Conn_01x03, J13 Conn_01x03, J14 Conn_01x20, J15 Conn_01x03, J16 Conn_01x03, J17 Hole, J18 Hole, J19 Hole, J2 Conn_01x02, J20 Hole, J21 Conn_01x02, J3 47346-0001, J4 Conn_01x04, J5 Conn_01x04, J6 20021121-00010C4LF, J7 Conn_01x02, J8 Conn_01x02, J9 Conn_01x02, Q1 NVTFS5C680NLTAG, Q2 NVTFS5C680NLTAG, U1 TMC2041-LA, U2 TMC2041-LA, U3 AP2112K-3.3, Y1 LFXTAL009678REEL

Commit message: add power header
Parts:
- added J22: Conn_01x06, Connector_PinSocket_2.54mm:PinSocket_1x06_P2.54mm_Vertical, symbol Connector_Generic:Conn_01x06
Connections:
- net +3V3: now also J22.3 (Pin_3), J22.4 (Pin_4)
- net +5V: now also J22.2 (Pin_2)
- net +VDC: now also J22.1 (Pin_1)
- net GND: now also J22.5 (Pin_5), J22.6 (Pin_6)
Other:
- moved on the sheet: J10, J11, J12, J13, J14, J15, J16, J2, J21, J4, J5, J9

Commit message: resolve a few issues in pcb design
Parts:
- removed IC1: MC7805BDTRKG, TO229P990X238-4N, symbol SamacSys_Parts:MC7805BDTRKG
- added C34, C35, C36: 10uF, Capacitor_SMD:C_0805_2012Metric, symbol Device:C
- added IC1: AP63205WU-7, SOT95P280X100-6N, symbol SamacSys_Parts:AP63205WU-7
- added L2, L3: 10uH, Inductor_SMD:L_0805_2012Metric, symbol Device:L
- C4: value 1uF -> 100nF
Connections:
- net +5V: now also C34.1, C35.1, C36.1, IC1.1 (FB), L2.1, L3.1; no longer C4.1
- net +VDC: now also IC1.2 (EN), IC1.3 (VIN)
- net GND: now also C34.2, C35.2, C36.2, IC1.4 (GND); no longer C4.2
- net SD_CS: now also IC2.51 (PA27)
- new net: C4.1, IC1.5 (SW), L2.2, L3.2
- new net: C4.2, IC1.6 (BST)
Other:
- moved on the sheet: C7

Commit message: pcb optimizations and fixes to v1 arduino package
Parts:
- removed J1: 47309-3351, 473093351, symbol SamacSys_Parts:47309-3351
- added J1: 47571-0001, 475710001, symbol SamacSys_Parts:47571-0001
Connections:
- net +3V3: now also J1.P4 (VDD)
- net GATE0: now also IC2.17 (PA08), J14.16 (Pin_16); no longer IC2.10 (PB07), J14.1 (Pin_1)
- net GATE1: now also IC2.18 (PA09), J14.17 (Pin_17); no longer IC2.11 (PB08), J14.2 (Pin_2)
- net GEN0: now also IC2.10 (PB07), J14.1 (Pin_1); no longer IC2.12 (PB09), J14.3 (Pin_3)
- net GEN1: now also IC2.11 (PB08), J14.2 (Pin_2); no longer IC2.13 (PA04), J14.4 (Pin_4)
- net GEN10: now also J14.11 (Pin_11); no longer J14.13 (Pin_13)
- net GEN11: now also J14.12 (Pin_12); no longer J14.14 (Pin_14)
- net GEN12: now also J14.13 (Pin_13); no longer J14.15 (Pin_15)
- net GEN13: now also J14.14 (Pin_14); no longer J14.16 (Pin_16)
- net GEN14: now also J14.15 (Pin_15); no longer J14.17 (Pin_17)
- net GEN2: now also IC2.12 (PB09), J14.3 (Pin_3); no longer IC2.14 (PA05), J14.5 (Pin_5)
- net GEN3: now also IC2.13 (PA04), J14.4 (Pin_4); no longer IC2.15 (PA06), J14.6 (Pin_6)
- net GEN4: now also IC2.14 (PA05), J14.5 (Pin_5); no longer IC2.16 (PA07), J14.7 (Pin_7)
- net GEN5: now also IC2.15 (PA06), J14.6 (Pin_6); no longer IC2.17 (PA08), J14.8 (Pin_8)
- net GEN6: now also IC2.16 (PA07), J14.7 (Pin_7); no longer IC2.18 (PA09), J14.9 (Pin_9)
- net GEN7: now also J14.8 (Pin_8); no longer J14.10 (Pin_10)
- net GEN8: now also J14.9 (Pin_9); no longer J14.11 (Pin_11)
- net GEN9: now also J14.10 (Pin_10); no longer J14.12 (Pin_12)
- net GND: now also J1.G1 (GND_1), J1.G2 (GND_2), J1.G3 (GND_3), J1.P6 (VSS)
- net MISO: now also J1.P7 (DAT0)
- net MOSI: now also J1.P3 (CMD)
- net SCK: now also J1.P5 (CLK)
- net SD_CS: now also J1.P2 (CD/DAT3)
- net SERVO0: now also IC2.31 (PA14), J14.18 (Pin_18), J16.1 (Pin_1); no longer IC2.35 (PA16), J13.1 (Pin_1), J14.20 (Pin_20)
- net SERVO2: now also IC2.35 (PA16), J13.1 (Pin_1), J14.20 (Pin_20); no longer IC2.31 (PA14), J14.18 (Pin_18), J16.1 (Pin_1)
Changed lines of the file:
@@
 $EndComp
 $Comp
-L SamacSys_Parts:47309-3351 J1
-U 1 1 5F283BC6
-P 19450 3300
-F 0 "J1" H 20100 3565 50  0000 C CNN
-F 1 "47309-3351" H 20100 3474 50  0000 C CNN
-F 2 "473093351" H 20600 3400 50  0001 L CNN
-F 3 "https://componentsearchengine.com/Datasheets/2/47309-3351.pdf" H 20600 3300 50  0001 L CNN
-F 4 "Molex 47309 Series 8 Way Right Angle Micro SD Memory Card Connector with Solder Termination" H 20600 3200 50  0001 L CNN "Description"
-F 5 "3.35" H 20600 3100 50  0001 L CNN "Height"
-F 6 "538-47309-3351" H 20600 3000 50  0001 L CNN "Mouser Part Number"
-F 7 "https://www.mouser.co.uk/ProductDetail/Molex/47309-3351?qs=7KFxWLW3pjpf5Z6T4AnH5Q%3D%3D" H 20600 2900 50  0001 L CNN "Mouser Price/Stock"
-F 8 "Molex" H 20600 2800 50  0001 L CNN "Manufacturer_Name"
-F 9 "47309-3351" H 20600 2700 50  0001 L CNN "Manufacturer_Part_Number"
-	1    19450 3300
-	1    0    0    -1
-$EndComp
-$Comp
 L power:+5V #PWR0107
 U 1 1 5F2A478B
@@
 	1    0    0    -1
 $EndComp
-Text Label 19350 3500 2    50   ~ 0
+Text Label 20900 3300 0    50   ~ 0
 MOSI
-Text Label 20850 3300 0    50   ~ 0
+Text Label 20900 3700 0    50   ~ 0
 MISO
 $Comp
 L power:GND #PWR0125
 U 1 1 5F4226D8
-P 19400 3850
-F 0 "#PWR0125" H 19400 3600 50  0001 C CNN
-F 1 "GND" H 19405 3677 50  0000 C CNN
-F 2 "" H 19400 3850 50  0001 C CNN
-F 3 "" H 19400 3850 50  0001 C CNN
-	1    19400 3850
+P 21200 3700
+F 0 "#PWR0125" H 21200 3450 50  0001 C CNN
+F 1 "GND" H 21205 3527 50  0000 C CNN
+F 2 "" H 21200 3700 50  0001 C CNN
+F 3 "" H 21200 3700 50  0001 C CNN
+	1    21200 3700
 	1    0    0    -1
 $EndComp
@@
 L power:+3.3V #PWR0126
 U 1 1 5F42DB4A
-P 19050 3450
-F 0 "#PWR0126" H 19050 3300 50  0001 C CNN
-F 1 "+3.3V" H 19065 3623 50  0000 C CNN
-F 2 "" H 19050 3450 50  0001 C CNN
-F 3 "" H 19050 3450 50  0001 C CNN
-	1    19050 3450
+P 21150 3250
+F 0 "#PWR0126" H 21150 3100 50  0001 C CNN
+F 1 "+3.3V" H 21165 3423 50  0000 C CNN
+F 2 "" H 21150 3250 50  0001 C CNN
+F 3 "" H 21150 3250 50  0001 C CNN
+	1    21150 3250
 	1    0    0    -1
 $EndComp
-Wire Wire Line
-	19450 3800 19400 3800
-Wire Wire Line
-	19400 3800 19400 3850
-Text Label 19050 3700 2    50   ~ 0
+Text Label 20900 3500 0    50   ~ 0
 SCK
 Wire Wire Line
-	19450 3700 19050 3700
-Wire Wire Line
-	19350 3500 19450 3500
+	20900 3300 20800 3300
 Wire Wire Line
-	20750 3300 20850 3300
-Text Label 19350 3200 2    50   ~ 0
+	20800 3700 20900 3700
+Text Label 19400 3900 2    50   ~ 0
 SD_CS
 Wire Wire Line
-	19050 3450 19050 3600
-Wire Wire Line
-	19050 3600 19450 3600
-Wire Wire Line
-	19350 3200 19350 3400
-Wire Wire Line
-	19350 3400 19450 3400
+	21150 3250 21150 3400
 $Comp
 L power:GND #PWR0102
 U 1 1 5F5BC76F
-P 21000 3650
-F 0 "#PWR0102" H 21000 3400 50  0001 C CNN
-F 1 "GND" H 21005 3477 50  0000 C CNN
-F 2 "" H 21000 3650 50  0001 C CNN
-F 3 "" H 21000 3650 50  0001 C CNN
-	1    21000 3650
+P 19150 3500
+F 0 "#PWR0102" H 19150 3250 50  0001 C CNN
+F 1 "GND" H 19155 3327 50  0000 C CNN
+F 2 "" H 19150 3500 50  0001 C CNN
+F 3 "" H 19150 3500 50  0001 C CNN
+	1    19150 3500
 	1    0    0    -1
 $EndComp
-Wire Wire Line
-	21000 3650 21000 3600
-Wire Wire Line
-	21000 3600 20750 3600
-Wire Wire Line
-	20750 3600 20750 3500
-Connection ~ 20750 3600
 $Comp
 L power:GND #PWR0103
@@
 Text Label 16000 4050 2    50   ~ 0
 GATE1
-Text Label 1300 3050 2    50   ~ 0
+Text Label 1750 4600 3    50   ~ 0
 GATE0
-Text Label 1300 3150 2    50   ~ 0
+Text Label 1850 4600 3    50   ~ 0
 GATE1
 Wire Wire Line
@@
 	1    0    0    -1
 $EndComp
-Text Label 21400 11000 0    50   ~ 0
+Text Label 21400 12300 0    50   ~ 0
 SERVO0
 Wire Wire Line
@@
 	1    0    0    -1
 $EndComp
-Text Label 21400 12300 0    50   ~ 0
+Text Label 21400 11000 0    50   ~ 0
 SERVO2
 Wire Wire Line
@@
 Wire Wire Line
 	21300 12500 21650 12500
-Text Label 3800 3450 0    50   ~ 0
+Text Label 3150 4600 3    50   ~ 0
 SERVO0
 Text Label 3250 4600 3    50   ~ 0
 SERVO1
-Text Label 3150 4600 3    50   ~ 0
+Text Label 3800 3450 0    50   ~ 0
 SERVO2
 Wire Wire Line
@@
 	1    0    0    -1
 $EndComp
-Text Label 1300 3450 2    50   ~ 0
+Text Label 1300 3250 2    50   ~ 0
 GEN2
-Text Label 1300 3550 2    50   ~ 0
+Text Label 1300 3350 2    50   ~ 0
 GEN3
-Text Label 1300 3650 2    50   ~ 0
+Text Label 1300 3450 2    50   ~ 0
 GEN4
-Text Label 1750 4600 3    50   ~ 0
+Text Label 1300 3550 2    50   ~ 0
 GEN5
-Text Label 1850 4600 3    50   ~ 0
+Text Label 1300 3650 2    50   ~ 0
 GEN6
 Text Label 1950 4600 3    50   ~ 0
@@
 Wire Wire Line
 	1950 4450 1950 4600
-Text Label 19950 13450 2    50   ~ 0
+Text Label 19950 13250 2    50   ~ 0
 SERVO0
 Wire Wire Line
@@
 Text Label 19950 13350 2    50   ~ 0
 SERVO1
-Text Label 19950 13250 2    50   ~ 0
+Text Label 19950 13450 2    50   ~ 0
 SERVO2
 Wire Wire Line
@@
 Wire Wire Line
 	1300 2950 1450 2950
-Text Label 19950 11950 2    50   ~ 0
+Text Label 19950 11750 2    50   ~ 0
 GEN2
-Text Label 19950 12050 2    50   ~ 0
+Text Label 19950 11850 2    50   ~ 0
 GEN3
-Text Label 19950 12150 2    50   ~ 0
+Text Label 19950 11950 2    50   ~ 0
 GEN4
-Text Label 19950 12250 2    50   ~ 0
+Text Label 19950 12050 2    50   ~ 0
 GEN5
-Text Label 19950 12350 2    50   ~ 0
+Text Label 19950 12150 2    50   ~ 0
 GEN6
 Wire Wire Line
@@
 Wire Wire Line
 	2050 4450 2050 4600
-Text Label 19950 12450 2    50   ~ 0
+Text Label 19950 12250 2    50   ~ 0
 GEN7
-Text Label 19950 12550 2    50   ~ 0
+Text Label 19950 12350 2    50   ~ 0
 GEN8
-Text Label 19950 12650 2    50   ~ 0
+Text Label 19950 12450 2    50   ~ 0
 GEN9
 Wire Wire Line
@@
 Wire Wire Line
 	20100 12750 19950 12750
-Text Label 19950 12850 2    50   ~ 0
+Text Label 19950 12650 2    50   ~ 0
 GEN11
-Text Label 19950 12950 2    50   ~ 0
+Text Label 19950 12750 2    50   ~ 0
 GEN12
-Text Label 19950 13050 2    50   ~ 0
+Text Label 19950 12850 2    50   ~ 0
 GEN13
 Wire Wire Line
@@
 Wire Wire Line
 	20100 13150 19950 13150
-Text Label 19950 13150 2    50   ~ 0
+Text Label 19950 12950 2    50   ~ 0
 GEN14
 Wire Wire Line
@@
 Wire Wire Line
 	20100 13450 19950 13450
-Text Label 19950 12750 2    50   ~ 0
+Text Label 19950 12550 2    50   ~ 0
 GEN10
 Wire Wire Line
@@
 Wire Wire Line
 	1300 2650 1450 2650
-Text Label 19950 11550 2    50   ~ 0
+Text Label 19950 13050 2    50   ~ 0
 GATE0
-Text Label 19950 11650 2    50   ~ 0
+Text Label 19950 13150 2    50   ~ 0
 GATE1
-Text Label 1300 3250 2    50   ~ 0
+Text Label 1300 3050 2    50   ~ 0
 GEN0
-Text Label 1300 3350 2    50   ~ 0
+Text Label 1300 3150 2    50   ~ 0
 GEN1
-Text Label 19950 11750 2    50   ~ 0
+Text Label 19950 11550 2    50   ~ 0
 GEN0
-Text Label 19950 11850 2    50   ~ 0
+Text Label 19950 11650 2    50   ~ 0
 GEN1
 Wire Notes Line
@@
 Wire Wire Line
 	3150 1200 3150 1350
+$Comp
+L SamacSys_Parts:47571-0001 J1
+U 1 1 5FCB4E4A
+P 19500 3300
+F 0 "J1" H 20150 3565 50  0000 C CNN
+F 1 "47571-0001" H 20150 3474 50  0000 C CNN
+F 2 "475710001" H 20650 3400 50  0001 L CNN
+F 3 "https://componentsearchengine.com/Datasheets/2/47571-0001.pdf" H 20650 3300 50  0001 L CNN
+F 4 "Memory Card Connectors ASSY FOR TFR HEADER HEADER W/DETECT PIN" H 20650 3200 50  0001 L CNN "Description"
+F 5 "2.3" H 20650 3100 50  0001 L CNN "Height"
+F 6 "538-47571-0001" H 20650 3000 50  0001 L CNN "Mouser Part Number"
+F 7 "https://www.mouser.co.uk/ProductDetail/Molex/47571-0001?qs=qM7ngqbhX5UTJOg9nqKLJQ%3D%3D" H 20650 2900 50  0001 L CNN "Mouser Price/Stock"
+F 8 "Molex" H 20650 2800 50  0001 L CNN "Manufacturer_Name"
+F 9 "47571-0001" H 20650 2700 50  0001 L CNN "Manufacturer_Part_Number"
+	1    19500 3300
+	1    0    0    -1
+$EndComp
+Wire Wire Line
+	20800 3400 21150 3400
+Wire Wire Line
+	19400 3900 19500 3900
+Wire Wire Line
+	20800 3500 20900 3500
+Wire Wire Line
+	20800 3600 21200 3600
+Wire Wire Line
+	21200 3600 21200 3700
+Wire Wire Line
+	19150 3500 19150 3300
+Wire Wire Line
+	19150 3300 19350 3300
+Wire Wire Line
+	19500 3400 19350 3400
+Wire Wire Line
+	19350 3400 19350 3300
+Connection ~ 19350 3300
+Wire Wire Line
+	19350 3300 19500 3300
+Wire Wire Line
+	19500 3500 19350 3500
+Wire Wire Line
+	19350 3500 19350 3400
+Connection ~ 19350 3400
 $EndSCHEMATC

Commit message: pcb v2 release
Parts:
- added R21: 100k, Resistor_SMD:R_0603_1608Metric, symbol Device:R
- added R22: 10k, Resistor_SMD:R_0603_1608Metric, symbol Device:R
Connections:
- net +VDC: now also R21.1
- net GND: now also R22.2
- net VSENSE: now reaches IC2.62 (PB01)
- net VSENSE: now also R21.2, R22.1
Other:
- moved on the sheet: C11, R2, U3
Changed lines of the file:
@@
 L Regulator_Linear:AP2112K-3.3 U3
 U 1 1 5F6EA1B6
-P 20950 8800
-F 0 "U3" H 20950 9142 50  0000 C CNN
-F 1 "AP2112K-3.3" H 20950 9051 50  0000 C CNN
-F 2 "Package_TO_SOT_SMD:SOT-23-5" H 20950 9125 50  0001 C CNN
-F 3 "https://www.diodes.com/assets/Datasheets/AP2112.pdf" H 20950 8900 50  0001 C CNN
-	1    20950 8800
+P 22050 8800
+F 0 "U3" H 22050 9142 50  0000 C CNN
+F 1 "AP2112K-3.3" H 22050 9051 50  0000 C CNN
+F 2 "Package_TO_SOT_SMD:SOT-23-5" H 22050 9125 50  0001 C CNN
+F 3 "https://www.diodes.com/assets/Datasheets/AP2112.pdf" H 22050 8900 50  0001 C CNN
+	1    22050 8800
 	1    0    0    -1
 $EndComp
@@
 L Device:R R2
 U 1 1 5F6FB56D
-P 20300 8900
-F 0 "R2" H 20370 8946 50  0000 L CNN
-F 1 "10k" H 20370 8855 50  0000 L CNN
-F 2 "Resistor_SMD:R_0603_1608Metric" V 20230 8900 50  0001 C CNN
-F 3 "~" H 20300 8900 50  0001 C CNN
-	1    20300 8900
+P 21400 8900
+F 0 "R2" H 21470 8946 50  0000 L CNN
+F 1 "10k" H 21470 8855 50  0000 L CNN
+F 2 "Resistor_SMD:R_0603_1608Metric" V 21330 8900 50  0001 C CNN
+F 3 "~" H 21400 8900 50  0001 C CNN
+	1    21400 8900
 	1    0    0    -1
 $EndComp
@@
 L Device:C C11
 U 1 1 5F6FF3D5
-P 21400 8900
-F 0 "C11" H 21515 8946 50  0000 L CNN
-F 1 "1uF" H 21515 8855 50  0000 L CNN
-F 2 "Capacitor_SMD:C_0603_1608Metric" H 21438 8750 50  0001 C CNN
-F 3 "~" H 21400 8900 50  0001 C CNN
-	1    21400 8900
+P 22500 8900
+F 0 "C11" H 22615 8946 50  0000 L CNN
+F 1 "1uF" H 22615 8855 50  0000 L CNN
+F 2 "Capacitor_SMD:C_0603_1608Metric" H 22538 8750 50  0001 C CNN
+F 3 "~" H 22500 8900 50  0001 C CNN
+	1    22500 8900
 	1    0    0    -1
 $EndComp
@@
 L power:GND #PWR0113
 U 1 1 5F705C53
-P 20950 9200
-F 0 "#PWR0113" H 20950 8950 50  0001 C CNN
-F 1 "GND" H 20955 9027 50  0000 C CNN
-F 2 "" H 20950 9200 50  0001 C CNN
-F 3 "" H 20950 9200 50  0001 C CNN
-	1    20950 9200
+P 22050 9200
+F 0 "#PWR0113" H 22050 8950 50  0001 C CNN
+F 1 "GND" H 22055 9027 50  0000 C CNN
+F 2 "" H 22050 9200 50  0001 C CNN
+F 3 "" H 22050 9200 50  0001 C CNN
+	1    22050 9200
 	1    0    0    -1
 $EndComp
@@
 L power:+5V #PWR0115
 U 1 1 5F70920F
-P 20500 8600
-F 0 "#PWR0115" H 20500 8450 50  0001 C CNN
-F 1 "+5V" H 20515 8773 50  0000 C CNN
-F 2 "" H 20500 8600 50  0001 C CNN
-F 3 "" H 20500 8600 50  0001 C CNN
-	1    20500 8600
-	1    0    0    -1
-$EndComp
-Wire Wire Line
-	20300 8750 20300 8700
-Wire Wire Line
-	20300 8700 20500 8700
-Wire Wire Line
-	20500 8600 20500 8700
-Connection ~ 20500 8700
-Wire Wire Line
-	20500 8700 20650 8700
-Wire Wire Line
-	20300 9050 20300 9100
-Wire Wire Line
-	20300 9100 20550 9100
-Wire Wire Line
-	20550 9100 20550 8800
-Wire Wire Line
-	20550 8800 20650 8800
-Wire Wire Line
-	20950 9100 20950 9150
-Wire Wire Line
-	21250 8700 21400 8700
-Wire Wire Line
-	21400 8700 21400 8750
+P 21600 8600
+F 0 "#PWR0115" H 21600 8450 50  0001 C CNN
+F 1 "+5V" H 21615 8773 50  0000 C CNN
+F 2 "" H 21600 8600 50  0001 C CNN
+F 3 "" H 21600 8600 50  0001 C CNN
+	1    21600 8600
+	1    0    0    -1
+$EndComp
+Wire Wire Line
+	21400 8750 21400 8700
+Wire Wire Line
+	21400 8700 21600 8700
+Wire Wire Line
+	21600 8600 21600 8700
+Connection ~ 21600 8700
+Wire Wire Line
+	21600 8700 21750 8700
+Wire Wire Line
+	21400 9050 21400 9100
+Wire Wire Line
+	21400 9100 21650 9100
+Wire Wire Line
+	21650 9100 21650 8800
+Wire Wire Line
+	21650 8800 21750 8800
+Wire Wire Line
+	22050 9100 22050 9150
+Wire Wire Line
+	22350 8700 22500 8700
+Wire Wire Line
+	22500 8700 22500 8750
 $Comp
 L power:+3.3V #PWR0117
 U 1 1 5F732118
-P 21550 8650
-F 0 "#PWR0117" H 21550 8500 50  0001 C CNN
-F 1 "+3.3V" H 21565 8823 50  0000 C CNN
-F 2 "" H 21550 8650 50  0001 C CNN
-F 3 "" H 21550 8650 50  0001 C CNN
-	1    21550 8650
-	1    0    0    -1
-$EndComp
-Wire Wire Line
-	21400 8700 21550 8700
-Wire Wire Line
-	21550 8700 21550 8650
-Connection ~ 21400 8700
-Wire Wire Line
-	21400 9050 21400 9150
-Wire Wire Line
-	21400 9150 20950 9150
-Connection ~ 20950 9150
-Wire Wire Line
-	20950 9150 20950 9200
+P 22650 8650
+F 0 "#PWR0117" H 22650 8500 50  0001 C CNN
+F 1 "+3.3V" H 22665 8823 50  0000 C CNN
+F 2 "" H 22650 8650 50  0001 C CNN
+F 3 "" H 22650 8650 50  0001 C CNN
+	1    22650 8650
+	1    0    0    -1
+$EndComp
+Wire Wire Line
+	22500 8700 22650 8700
+Wire Wire Line
+	22650 8700 22650 8650
+Connection ~ 22500 8700
+Wire Wire Line
+	22500 9050 22500 9150
+Wire Wire Line
+	22500 9150 22050 9150
+Connection ~ 22050 9150
+Wire Wire Line
+	22050 9150 22050 9200
 $Comp
 L Device:C C5
@@
 	19350 3500 19350 3400
 Connection ~ 19350 3400
+$Comp
+L Device:R R21
+U 1 1 5FD5544D
+P 19950 8550
+F 0 "R21" H 20020 8596 50  0000 L CNN
+F 1 "100k" H 20020 8505 50  0000 L CNN
+F 2 "Resistor_SMD:R_0603_1608Metric" V 19880 8550 50  0001 C CNN
+F 3 "~" H 19950 8550 50  0001 C CNN
+	1    19950 8550
+	1    0    0    -1
+$EndComp
+$Comp
+L power:+VDC #PWR0171
+U 1 1 5FD96175
+P 19950 8300
+F 0 "#PWR0171" H 19950 8200 50  0001 C CNN
+F 1 "+VDC" H 19950 8575 50  0000 C CNN
+F 2 "" H 19950 8300 50  0001 C CNN
+F 3 "" H 19950 8300 50  0001 C CNN
+	1    19950 8300
+	1    0    0    -1
+$EndComp
+$Comp
+L Device:R R22
+U 1 1 5FE17BC1
+P 19950 8950
+F 0 "R22" H 20020 8996 50  0000 L CNN
+F 1 "10k" H 20020 8905 50  0000 L CNN
+F 2 "Resistor_SMD:R_0603_1608Metric" V 19880 8950 50  0001 C CNN
+F 3 "~" H 19950 8950 50  0001 C CNN
+	1    19950 8950
+	1    0    0    -1
+$EndComp
+$Comp
+L power:GND #PWR0172
+U 1 1 5FE58697
+P 19950 9200
+F 0 "#PWR0172" H 19950 8950 50  0001 C CNN
+F 1 "GND" H 19955 9027 50  0000 C CNN
+F 2 "" H 19950 9200 50  0001 C CNN
+F 3 "" H 19950 9200 50  0001 C CNN
+	1    19950 9200
+	1    0    0    -1
+$EndComp
+Wire Wire Line
+	19950 8300 19950 8400
+Wire Wire Line
+	19950 8700 19950 8750
+Wire Wire Line
+	19950 9100 19950 9200
+Text Label 19800 8750 2    50   ~ 0
+VSENSE
+Wire Wire Line
+	19800 8750 19950 8750
+Connection ~ 19950 8750
+Wire Wire Line
+	19950 8750 19950 8800
+Text Label 2050 1200 1    50   ~ 0
+VSENSE
 $EndSCHEMATC
