File: pcb/KiCad Schematic.sch (KiCad schematic (older format))
At the start: 96 parts, among them IC1 AP63205WU-7, IC2 ATSAMD51J19A-MU, J1 47571-0001, J10 Conn_01x04, J11 Conn_01x04, J12 Conn_01x03, J13 Conn_01x03, J14 Conn_01x20, J15 Conn_01x03, J16 Conn_01x03, J17 Hole, J18 Hole, J19 Hole, J2 Conn_01x02, J20 Hole, J21 Conn_01x02, J22 Conn_01x06, J3 47346-0001, J4 Conn_01x04, J5 Conn_01x04, J6 20021121-00010C4LF, J7 Conn_01x02, J8 Conn_01x02, J9 Conn_01x02, Q1 NVTFS5C680NLTAG, Q2 NVTFS5C680NLTAG, U1 TMC2041-LA, U2 TMC2041-LA, U3 AP2112K-3.3, Y1 LFXTAL009678REEL

Commit message: arduino version bump
Parts:
- added D5: CGRTS4004-HF, Diode_SMD:D_SOD-123F, symbol Device:D
Connections:
- net +3V3: now also C36.1
- net +5V: no longer C36.1
- net +VDC: now also D5.2 (A); no longer C7.1, IC1.2 (EN), IC1.3 (VIN)
- new net: C7.1, D5.1 (K), IC1.2 (EN), IC1.3 (VIN)
Other:
- moved on the sheet: C11, R2, U3
Changed lines of the file:
@@
 L Regulator_Linear:AP2112K-3.3 U3
 U 1 1 5F6EA1B6
-P 22050 8800
-F 0 "U3" H 22050 9142 50  0000 C CNN
-F 1 "AP2112K-3.3" H 22050 9051 50  0000 C CNN
-F 2 "Package_TO_SOT_SMD:SOT-23-5" H 22050 9125 50  0001 C CNN
-F 3 "https://www.diodes.com/assets/Datasheets/AP2112.pdf" H 22050 8900 50  0001 C CNN
-	1    22050 8800
+P 21450 8650
+F 0 "U3" H 21450 8992 50  0000 C CNN
+F 1 "AP2112K-3.3" H 21450 8901 50  0000 C CNN
+F 2 "Package_TO_SOT_SMD:SOT-23-5" H 21450 8975 50  0001 C CNN
+F 3 "https://www.diodes.com/assets/Datasheets/AP2112.pdf" H 21450 8750 50  0001 C CNN
+	1    21450 8650
 	1    0    0    -1
 $EndComp
@@
 L Device:R R2
 U 1 1 5F6FB56D
-P 21400 8900
-F 0 "R2" H 21470 8946 50  0000 L CNN
-F 1 "10k" H 21470 8855 50  0000 L CNN
-F 2 "Resistor_SMD:R_0603_1608Metric" V 21330 8900 50  0001 C CNN
-F 3 "~" H 21400 8900 50  0001 C CNN
-	1    21400 8900
+P 20800 8750
+F 0 "R2" H 20870 8796 50  0000 L CNN
+F 1 "10k" H 20870 8705 50  0000 L CNN
+F 2 "Resistor_SMD:R_0603_1608Metric" V 20730 8750 50  0001 C CNN
+F 3 "~" H 20800 8750 50  0001 C CNN
+	1    20800 8750
 	1    0    0    -1
 $EndComp
@@
 L Device:C C11
 U 1 1 5F6FF3D5
-P 22500 8900
-F 0 "C11" H 22615 8946 50  0000 L CNN
-F 1 "1uF" H 22615 8855 50  0000 L CNN
-F 2 "Capacitor_SMD:C_0603_1608Metric" H 22538 8750 50  0001 C CNN
-F 3 "~" H 22500 8900 50  0001 C CNN
-	1    22500 8900
+P 21900 8750
+F 0 "C11" H 22015 8796 50  0000 L CNN
+F 1 "1uF" H 22015 8705 50  0000 L CNN
+F 2 "Capacitor_SMD:C_0603_1608Metric" H 21938 8600 50  0001 C CNN
+F 3 "~" H 21900 8750 50  0001 C CNN
+	1    21900 8750
 	1    0    0    -1
 $EndComp
@@
 L power:GND #PWR0113
 U 1 1 5F705C53
-P 22050 9200
-F 0 "#PWR0113" H 22050 8950 50  0001 C CNN
-F 1 "GND" H 22055 9027 50  0000 C CNN
-F 2 "" H 22050 9200 50  0001 C CNN
-F 3 "" H 22050 9200 50  0001 C CNN
-	1    22050 9200
+P 21450 9050
+F 0 "#PWR0113" H 21450 8800 50  0001 C CNN
+F 1 "GND" H 21455 8877 50  0000 C CNN
+F 2 "" H 21450 9050 50  0001 C CNN
+F 3 "" H 21450 9050 50  0001 C CNN
+	1    21450 9050
 	1    0    0    -1
 $EndComp
@@
 L power:+5V #PWR0115
 U 1 1 5F70920F
-P 21600 8600
-F 0 "#PWR0115" H 21600 8450 50  0001 C CNN
-F 1 "+5V" H 21615 8773 50  0000 C CNN
-F 2 "" H 21600 8600 50  0001 C CNN
-F 3 "" H 21600 8600 50  0001 C CNN
-	1    21600 8600
-	1    0    0    -1
-$EndComp
-Wire Wire Line
-	21400 8750 21400 8700
-Wire Wire Line
-	21400 8700 21600 8700
-Wire Wire Line
-	21600 8600 21600 8700
-Connection ~ 21600 8700
-Wire Wire Line
-	21600 8700 21750 8700
-Wire Wire Line
-	21400 9050 21400 9100
-Wire Wire Line
-	21400 9100 21650 9100
-Wire Wire Line
-	21650 9100 21650 8800
-Wire Wire Line
-	21650 8800 21750 8800
-Wire Wire Line
-	22050 9100 22050 9150
-Wire Wire Line
-	22350 8700 22500 8700
-Wire Wire Line
-	22500 8700 22500 8750
+P 21000 8450
+F 0 "#PWR0115" H 21000 8300 50  0001 C CNN
+F 1 "+5V" H 21015 8623 50  0000 C CNN
+F 2 "" H 21000 8450 50  0001 C CNN
+F 3 "" H 21000 8450 50  0001 C CNN
+	1    21000 8450
+	1    0    0    -1
+$EndComp
+Wire Wire Line
+	20800 8600 20800 8550
+Wire Wire Line
+	20800 8550 21000 8550
+Wire Wire Line
+	21000 8450 21000 8550
+Connection ~ 21000 8550
+Wire Wire Line
+	21000 8550 21150 8550
+Wire Wire Line
+	20800 8900 20800 8950
+Wire Wire Line
+	20800 8950 21050 8950
+Wire Wire Line
+	21050 8950 21050 8650
+Wire Wire Line
+	21050 8650 21150 8650
+Wire Wire Line
+	21450 8950 21450 9000
+Wire Wire Line
+	21750 8550 21900 8550
+Wire Wire Line
+	21900 8550 21900 8600
 $Comp
 L power:+3.3V #PWR0117
 U 1 1 5F732118
-P 22650 8650
-F 0 "#PWR0117" H 22650 8500 50  0001 C CNN
-F 1 "+3.3V" H 22665 8823 50  0000 C CNN
-F 2 "" H 22650 8650 50  0001 C CNN
-F 3 "" H 22650 8650 50  0001 C CNN
-	1    22650 8650
-	1    0    0    -1
-$EndComp
-Wire Wire Line
-	22500 8700 22650 8700
-Wire Wire Line
-	22650 8700 22650 8650
-Connection ~ 22500 8700
-Wire Wire Line
-	22500 9050 22500 9150
-Wire Wire Line
-	22500 9150 22050 9150
-Connection ~ 22050 9150
-Wire Wire Line
-	22050 9150 22050 9200
+P 22450 8500
+F 0 "#PWR0117" H 22450 8350 50  0001 C CNN
+F 1 "+3.3V" H 22465 8673 50  0000 C CNN
+F 2 "" H 22450 8500 50  0001 C CNN
+F 3 "" H 22450 8500 50  0001 C CNN
+	1    22450 8500
+	1    0    0    -1
+$EndComp
+Wire Wire Line
+	21900 8900 21900 9000
+Wire Wire Line
+	21900 9000 21450 9000
+Connection ~ 21450 9000
+Wire Wire Line
+	21450 9000 21450 9050
 $Comp
 L Device:C C5
@@
 L power:+VDC #PWR0138
 U 1 1 6003EFAA
-P 18950 6900
-F 0 "#PWR0138" H 18950 6800 50  0001 C CNN
-F 1 "+VDC" H 18950 7175 50  0000 C CNN
-F 2 "" H 18950 6900 50  0001 C CNN
-F 3 "" H 18950 6900 50  0001 C CNN
-	1    18950 6900
+P 18950 6800
+F 0 "#PWR0138" H 18950 6700 50  0001 C CNN
+F 1 "+VDC" H 18950 7075 50  0000 C CNN
+F 2 "" H 18950 6800 50  0001 C CNN
+F 3 "" H 18950 6800 50  0001 C CNN
+	1    18950 6800
 	1    0    0    -1
 $EndComp
@@
 	21750 7200 22150 7200
 Connection ~ 21750 7200
-$Comp
-L Device:C C36
-U 1 1 6014CE08
-P 22550 7350
-F 0 "C36" H 22665 7396 50  0000 L CNN
-F 1 "10uF" H 22665 7305 50  0000 L CNN
-F 2 "Capacitor_SMD:C_0805_2012Metric" H 22588 7200 50  0001 C CNN
-F 3 "~" H 22550 7350 50  0001 C CNN
-	1    22550 7350
-	1    0    0    -1
-$EndComp
-Wire Wire Line
-	22150 7200 22550 7200
 Connection ~ 22150 7200
 Wire Wire Line
-	22550 7200 22700 7200
-Wire Wire Line
 	22700 7200 22700 7100
-Connection ~ 22550 7200
-Wire Wire Line
-	22550 7500 22550 7550
-Wire Wire Line
-	22550 7550 22150 7550
 Wire Wire Line
 	21750 7550 21750 7500
@@
 	1    0    0    -1
 $EndComp
-Wire Wire Line
-	18950 6900 18950 7300
 Wire Wire Line
 	18950 7300 19100 7300
@@
 Text Label 2050 1200 1    50   ~ 0
 VSENSE
+$Comp
+L Device:D D5
+U 1 1 6023B05C
+P 18950 7050
+F 0 "D5" H 18950 6834 50  0000 C CNN
+F 1 "CGRTS4004-HF" H 18950 6925 50  0000 C CNN
+F 2 "Diode_SMD:D_SOD-123F" H 18950 7050 50  0001 C CNN
+F 3 "~" H 18950 7050 50  0001 C CNN
+	1    18950 7050
+	0    -1   -1   0
+$EndComp
+Wire Wire Line
+	18950 6800 18950 6900
+Wire Wire Line
+	18950 7200 18950 7300
+$Comp
+L Device:C C36
+U 1 1 60407D4F
+P 22300 8750
+F 0 "C36" H 22415 8796 50  0000 L CNN
+F 1 "10uF" H 22415 8705 50  0000 L CNN
+F 2 "Capacitor_SMD:C_0805_2012Metric" H 22338 8600 50  0001 C CNN
+F 3 "~" H 22300 8750 50  0001 C CNN
+	1    22300 8750
+	1    0    0    -1
+$EndComp
+Wire Wire Line
+	22150 7200 22700 7200
+Wire Wire Line
+	22300 8900 22300 9000
+Wire Wire Line
+	22300 9000 21900 9000
+Connection ~ 21900 9000
+Wire Wire Line
+	21900 8550 22300 8550
+Wire Wire Line
+	22300 8550 22300 8600
+Connection ~ 21900 8550
+Wire Wire Line
+	22300 8550 22450 8550
+Wire Wire Line
+	22450 8550 22450 8500
+Connection ~ 22300 8550
 $EndSCHEMATC
